File: eGatewayShield/eGatewayShield.sch (EAGLE design)
At the start: 17 parts, among them SW1 SPST_TACT-EVQQ2, U1 ATMEGA328P_TQFP, U2 RFM69HW, X1 RASPI_BOARD_B+#_F, Y1 16MHZ

Commit message: Add Backup files from old smart home project
Parts:
- removed ANT: LSP13, solpad:LSP13
- removed C1, C2, C3: 0.1uF, SparkFun-Capacitors:CAP0603-CAP
- removed FTDI: (no value), pinhead:PINHD-1X5
- removed LED1, LED2: (no value), adafruit:LEDCHIPLED_0603
- removed R1: (no value), SparkFun-Resistors:RESISTOR0603-RES
- removed R2, R3: 1K, SparkFun-Resistors:RESISTOR0603-RES
- removed SPI: (no value), pinhead:PINHD-1X6
- removed SW1: SPST_TACT-EVQQ2, adafruit:SPST_TACT-EVQQ2
- removed U1: ATMEGA328P_TQFP, SparkFun-DigitalIC:ATMEGA328P_TQFP
- removed U2: RFM69HW, SparkFun-RF:RFM69HW
- removed Y1: 16MHZ, SparkFun-FreqCtrl:RESONATOR16MHZ
- added U$2: MOTEINO_R4_MODULEUSING_SQ_POST_PINS, MoteinoR4Mod:MOTEINO_R4_MODULEUSING_SQ_POST_PINS
Connections:
- removed net A4/SDA: I2C.4, U1.PC4(ADC4/SDA)
- removed net A5/SCL: I2C.3, U1.PC5(ADC5/SCL)
- removed net ANT: ANT.MP, U2.ANT
- removed net D10/SS: SPI.6, U1.PB2(SS/OC1B), U2.NSS
- removed net D11/MOSI: SPI.5, U1.PB3(MOSI/OC2), U2.MOSI
- removed net D12/MISO: SPI.4, U1.PB4(MISO), U2.MISO
- removed net D13/SCK: SPI.3, U1.PB5(SCK), U2.SCK
- removed net D2: U1.PD2(INT0), U2.DIO0
- removed net D3: U1.PD3(INT1)
- removed net DTR: C2.1
- removed net N$1: LED1.C, R2.1
- removed net N$2: LED2.C, R3.1
- removed net N$7: C1.1, U1.AREF
- removed net RESET: C2.2, FTDI.5, R1.1, SW1.S, SW1.S1, U1.PC6(/RESET)
- removed net RX: FTDI.4, R2.2, U1.PD0(RXD), X1.TXD
- removed net TX: FTDI.3, R3.2, U1.PD1(TXD), X1.RXD
- removed net XTAL1: U1.PB6(XTAL1/TOSC1), Y1.1
- removed net XTAL2: U1.PB7(XTAL2/TOSC2), Y1.3
- new net 5V: U$2.PWR, X1.5V0A
- new net RXI: U$2.D1_TX, X1.TXD
- new net SCL: I2C.2, X1.SCL
- new net SDA: I2C.1, X1.SDA
- new net TXO: U$2.D0_RX, X1.RXD
- net 3.3V: now also I2C.4, U$2.3.3V@1; no longer C3.1, FTDI.2, I2C.2, LED1.A, LED2.A, R1.2, SPI.2, U1.AVCC, U1.VCC@4, U1.VCC@6, U2.3.3V
- net GND: now also I2C.3, U$2.GND@1, U$2.GND@2; no longer C1.2, C3.2, FTDI.1, I2C.1, SPI.1, SW1.P, SW1.P1, U1.AGND, U1.GND@3, U1.GND@5, U2.GND@1, Y1.2
Other:
- moved on the sheet: I2C
